File: PCB/PCB.kicad_pcb (KiCad board)
At the start: 2 copper layers, 66.3 x 47.8 mm, 38 parts, among them J1 Conn_01x03_Pin, J2 Conn_01x04_Pin, J3 Conn_01x04_Socket, J4 Conn_01x05_Socket, Q1 BC807, U1 Pico, U2 HX711

Commit message: PCB V1.0 orderd
Parts:
- added H1: MountingHole, MountingHole:MountingHole_3.2mm_M3_DIN965, F.Cu at (78.6, 39.6)
- added H2: MountingHole, MountingHole:MountingHole_3.2mm_M3_DIN965, F.Cu at (78.6, 81.2)
- added H3: MountingHole, MountingHole:MountingHole_3.2mm_M3_DIN965, F.Cu at (138.7, 81.1)
- added H4: MountingHole, MountingHole:MountingHole_3.2mm_M3_DIN965, F.Cu at (138.7, 39.6)
- moved C2 17.8 mm to (107.9, 70.8)
- moved R2 12.4 mm to (118.8, 70.8)
- moved R4 12.3 mm to (105.0, 70.8)
- moved JP2 9.99 mm to (132.6, 62.5)
- moved R5 9.99 mm to (113.4, 70.8)
- moved TP6 9.99 mm to (106.3, 48.4)
- moved U2 9.99 mm to (140.3, 72.8)
- moved JP1 9.99 mm to (137.7, 62.4)
- moved TP13 9.99 mm to (106.3, 59.7)
- moved TP9 9.99 mm to (106.3, 44.1)
- moved C3 9.99 mm to (110.7, 70.8)
- moved C4 9.99 mm to (86.1, 42.4)
- moved C5 9.99 mm to (88.8, 42.3)
- moved C7 9.99 mm to (94.5, 42.4)
- moved C8 9.99 mm to (97.3, 42.3)
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Connections:
- C1 pad 1: /encoder_b -> /encoder_a
- C2 pad 1: /encoder_a -> /encoder_b
- J4 pad 3: /encoder_b -> /encoder_a
- J4 pad 4: /encoder_a -> /encoder_b
- JP1 pad 1: Net-(J2-Pin_3) -> Net-(J2-Pin_4)
- JP2 pad 1: Net-(J2-Pin_3) -> Net-(J2-Pin_4)
- JP3 pad 1: Net-(J2-Pin_4) -> Net-(J2-Pin_3)
- JP4 pad 1: Net-(J2-Pin_4) -> Net-(J2-Pin_3)
- R3 pad 2: /encoder_b -> /encoder_a
- R4 pad 2: /encoder_a -> /encoder_b
- TP13 pad 1: /encoder_b -> unconnected-(TP13-Pad1)
- TP14 pad 1: /encoder_a -> unconnected-(TP14-Pad1)
- U1 pad 16: /encoder_a -> /encoder_b
- U1 pad 17: /encoder_b -> /encoder_a
Routing:
- net Net-(J2-Pin_4): track 14.4 -> 25.7 mm
- net Net-(J2-Pin_3): track 25.0 -> 14.5 mm, vias 1 -> 0
- net /LCD_SDA: track 39.7 -> 43.8 mm
- net +5V: track 143.1 -> 139.1 mm
- net /encoder_a: track 38.3 -> 35.8 mm
- net Net-(J2-Pin_2): track 13.6 -> 12.8 mm
- net /Relay: track 12.5 -> 13.4 mm
- net Net-(J2-Pin_1): track 13.7 -> 12.8 mm
- net GND: vias 50 -> 62
