File: PCB/PCB.kicad_sch (KiCad schematic)
At the start: 20 parts, among them J1 Conn_01x03_Pin, J2 Conn_01x04_Pin, Q1 BC807, U1 Pico, U2 HX711

Commit message: schaltplan fertig
Parts:
- added C1, C2, C3: 100n, Capacitor_SMD:C_0603_1608Metric_Pad1.08x0.95mm_HandSolder, symbol Device:C
- added J3: Conn_01x04_Socket, Connector_PinHeader_2.54mm:PinHeader_1x04_P2.54mm_Vertical, symbol Connector:Conn_01x04_Socket
- added J4: Conn_01x05_Socket, Connector_PinHeader_2.54mm:PinHeader_1x05_P2.54mm_Vertical, symbol Connector:Conn_01x05_Socket
- added R1, R2, R3, R4, R5, R6: 3.3k, Resistor_SMD:R_0603_1608Metric_Pad0.98x0.95mm_HandSolder, symbol Device:R
- added TP12, TP13, TP14, TP15, TP16: TestPoint, TestPoint:TestPoint_Pad_D2.0mm, symbol Connector:TestPoint
Connections:
- net +5V: now also J3.2 (Pin_2), J4.2 (Pin_2), R1.1, R2.1, R3.1, R4.1, R5.1
- net GND: now also C1.2, C2.2, C3.2, J3.1 (Pin_1), J4.1 (Pin_1)
- net HX711_SCK: now also U1.9 (GPIO6)
- net HX/11_DT: now also U1.7 (GPIO5)
- net Relay_3.3: now reaches TP7.1, U1.5 (GPIO3)
- net Relay_3.3: now also R6.1; no longer Q1.1 (B)
- net LCD_SDA: now reaches U1.11 (GPIO8)
- net LCD_SDA: now also J3.3 (Pin_3), R1.2, TP15.1
- net LCD_SCL: now reaches U1.12 (GPIO9)
- net LCD_SCL: now also J3.4 (Pin_4), R2.2, TP16.1
- net encoder_button: now reaches U1.15 (GPIO11)
- net encoder_button: now also C3.1, J4.5 (Pin_5), R5.2, TP12.1
- net encoder_a: now reaches U1.16 (GPIO12)
- net encoder_a: now also C1.1, J4.3 (Pin_3), R3.2, TP14.1
- net encoder_b: now reaches U1.17 (GPIO13)
- net encoder_b: now also C2.1, J4.4 (Pin_4), R4.2, TP13.1
- new net: Q1.1 (B), R6.2
Other:
- moved on the sheet: TP1, TP2, TP3, TP4, TP5, U1
