File: PCB/PCB.kicad_sch (KiCad schematic)
At the start: 38 parts, among them J1 Conn_01x03_Pin, J2 Conn_01x04_Pin, J3 Conn_01x04_Socket, J4 Conn_01x05_Socket, Q1 BC807, U1 Pico, U2 HX711

Commit message: PCB V1.0 orderd
Parts:
- added H1, H2, H3, H4: MountingHole, MountingHole:MountingHole_3.2mm_M3_DIN965, symbol Mechanical:MountingHole
Connections:
- net encoder_a: now also C1.1, J4.3 (Pin_3), R3.2, U1.17 (GPIO13); no longer C2.1, J4.4 (Pin_4), R4.2, TP14.1, U1.16 (GPIO12)
- net encoder_b: now also C2.1, J4.4 (Pin_4), R4.2, U1.16 (GPIO12); no longer C1.1, J4.3 (Pin_3), R3.2, TP13.1, U1.17 (GPIO13)
- net at JP1.1 (A), JP2.1 (A): now also J2.4 (Pin_4); no longer J2.3 (Pin_3)
- net at JP3.1 (A), JP4.1 (A): now also J2.3 (Pin_3); no longer J2.4 (Pin_4)
Other:
- moved on the sheet: JP1, JP2, JP3, JP4, TP4, TP5, U1
