File: PCB/_autosave-PCB.kicad_pcb (KiCad board)
At the start: 2 copper layers, 66.3 x 47.8 mm, 38 parts, among them J1 Conn_01x03_Pin, J2 Conn_01x04_Pin, J3 Conn_01x04_Socket, J4 Conn_01x05_Socket, Q1 BC807, U1 Pico, U2 HX711

Commit message: PCB fertig
Parts:
- moved C1 8.47 mm to (90.8, 75.7)
- moved C2 8.41 mm to (99.3, 75.7)
- moved J2 4.42 mm to (115.2, 82.4)
- moved R3 3.03 mm to (93.5, 75.7)
- moved R1 2.72 mm to (107.4, 75.7)
- moved R2 2.72 mm to (110.1, 75.7)
- moved R4 2.56 mm to (96.3, 75.7)
Connections:
- C1 pad 1: /encoder_b -> /encoder_a
- C2 pad 1: /encoder_a -> /encoder_b
- J4 pad 3: /encoder_b -> /encoder_a
- J4 pad 4: /encoder_a -> /encoder_b
- JP1 pad 1: Net-(J2-Pin_3) -> Net-(J2-Pin_4)
- JP2 pad 1: Net-(J2-Pin_3) -> Net-(J2-Pin_4)
- JP3 pad 1: Net-(J2-Pin_4) -> Net-(J2-Pin_3)
- JP4 pad 1: Net-(J2-Pin_4) -> Net-(J2-Pin_3)
- R3 pad 2: /encoder_b -> /encoder_a
- R4 pad 2: /encoder_a -> /encoder_b
- TP13 pad 1: /encoder_b -> unconnected-(TP13-Pad1)
- TP14 pad 1: /encoder_a -> unconnected-(TP14-Pad1)
- U1 pad 16: /encoder_a -> /encoder_b
- U1 pad 17: /encoder_b -> /encoder_a
Routing:
- net Net-(J2-Pin_4): track 14.4 -> 25.7 mm
- net Net-(J2-Pin_3): track 25.0 -> 14.7 mm, vias 1 -> 0
- net /encoder_b: track 38.9 -> 47.5 mm
- net /LCD_SDA: track 39.7 -> 43.8 mm
- net /encoder_a: track 38.3 -> 40.1 mm
- net +5V: track 143.1 -> 144.0 mm
- net Net-(J2-Pin_2): track 13.6 -> 12.8 mm
- net Net-(J2-Pin_1): track 13.7 -> 12.8 mm
- net GND: vias 50 -> 61
